Commit message: Automate URDF parsing using .env configuration

File: public/urdf/sophia_v2.urdf (robot description, URDF)
Before this commit: robot sophia_hexapod, 26 links, 25 joints
Links:
- link base_link: mass 0.5 -> 0.402; geometry collision cylinder length=0.055 radius=0.06; visual cylinder length=0.055 radius=0.06
- link lb_base_motor_link: mass 0.01 -> 0.001
- link lb_coxa_link: mass 0.05 -> 0.006; geometry collision box size=0.035 0.03 0.03; visual box size=0.035 0.03 0.03
- link lb_femur_link: mass 0.1 -> 0.033; geometry collision box size=0.045 0.025 0.025; visual box size=0.045 0.025 0.025
- link lb_tibia_link: mass 0.08 -> 0.009; geometry collision box size=0.08249999999999999 0.015 0.015; collision sphere radius=0.0075
- link lf_base_motor_link: mass 0.01 -> 0.001
- link lf_coxa_link: mass 0.05 -> 0.006; geometry collision box size=0.035 0.03 0.03; visual box size=0.035 0.03 0.03
- link lf_femur_link: mass 0.1 -> 0.033; geometry collision box size=0.045 0.025 0.025; visual box size=0.045 0.025 0.025
- link lf_tibia_link: mass 0.08 -> 0.009; geometry collision box size=0.08249999999999999 0.015 0.015; collision sphere radius=0.0075
- link lm_base_motor_link: mass 0.01 -> 0.001
- link lm_coxa_link: mass 0.05 -> 0.006; geometry collision box size=0.035 0.03 0.03; visual box size=0.035 0.03 0.03
- link lm_femur_link: mass 0.1 -> 0.033; geometry collision box size=0.045 0.025 0.025; visual box size=0.045 0.025 0.025
- link lm_tibia_link: mass 0.08 -> 0.009; geometry collision box size=0.08249999999999999 0.015 0.015; collision sphere radius=0.0075
- link rb_base_motor_link: mass 0.01 -> 0.001
- link rb_coxa_link: mass 0.05 -> 0.006; geometry collision box size=0.035 0.03 0.03; visual box size=0.035 0.03 0.03
- link rb_femur_link: mass 0.1 -> 0.033; geometry collision box size=0.045 0.025 0.025; visual box size=0.045 0.025 0.025
- link rb_tibia_link: mass 0.08 -> 0.009; geometry collision box size=0.08249999999999999 0.015 0.015; collision sphere radius=0.0075
- link rf_base_motor_link: mass 0.01 -> 0.001
- link rf_coxa_link: mass 0.05 -> 0.006; geometry collision box size=0.035 0.03 0.03; visual box size=0.035 0.03 0.03
- link rf_femur_link: mass 0.1 -> 0.033; geometry collision box size=0.045 0.025 0.025; visual box size=0.045 0.025 0.025
- link rf_tibia_link: mass 0.08 -> 0.009; geometry collision box size=0.08249999999999999 0.015 0.015; collision sphere radius=0.0075
- link rm_base_motor_link: mass 0.01 -> 0.001
- link rm_coxa_link: mass 0.05 -> 0.006; geometry collision box size=0.035 0.03 0.03; visual box size=0.035 0.03 0.03
- link rm_femur_link: mass 0.1 -> 0.033; geometry collision box size=0.045 0.025 0.025; visual box size=0.045 0.025 0.025
- link rm_tibia_link: mass 0.08 -> 0.009; geometry collision box size=0.08249999999999999 0.015 0.015; collision sphere radius=0.0075
Joints:
- joint lb_coxa_joint: limit lower=-1.0 upper=1.0 effort=5.0 velocity=12 -> lower=-3.141592653589793 upper=3.141592653589793 effort=0.2 velocity=11.6
- joint lb_coxa_link_to_lb_femur_link: limit lower=-1.85 upper=1.57 effort=5.0 velocity=12 -> lower=-3.141592653589793 upper=3.141592653589793 effort=0.2 velocity=11.6
- joint lb_femur_link_to_lb_tibia_link: limit lower=-2.0 upper=2.75 effort=5.0 velocity=12 -> lower=-3.141592653589793 upper=3.141592653589793 effort=0.2 velocity=11.6
- joint lf_coxa_joint: limit lower=-1.0 upper=1.0 effort=5.0 velocity=12 -> lower=-3.141592653589793 upper=3.141592653589793 effort=0.2 velocity=11.6
- joint lf_coxa_link_to_lf_femur_link: limit lower=-1.85 upper=1.57 effort=5.0 velocity=12 -> lower=-3.141592653589793 upper=3.141592653589793 effort=0.2 velocity=11.6
- joint lf_femur_link_to_lf_tibia_link: limit lower=-2.0 upper=2.75 effort=5.0 velocity=12 -> lower=-3.141592653589793 upper=3.141592653589793 effort=0.2 velocity=11.6
- joint lm_coxa_joint: limit lower=-1.0 upper=1.0 effort=5.0 velocity=12 -> lower=-3.141592653589793 upper=3.141592653589793 effort=0.2 velocity=11.6
- joint lm_coxa_link_to_lm_femur_link: limit lower=-1.85 upper=1.57 effort=5.0 velocity=12 -> lower=-3.141592653589793 upper=3.141592653589793 effort=0.2 velocity=11.6
- joint lm_femur_link_to_lm_tibia_link: limit lower=-2.0 upper=2.75 effort=5.0 velocity=12 -> lower=-3.141592653589793 upper=3.141592653589793 effort=0.2 velocity=11.6
- joint rb_coxa_joint: limit lower=-1.0 upper=1.0 effort=5.0 velocity=12 -> lower=-3.141592653589793 upper=3.141592653589793 effort=0.2 velocity=11.6
- joint rb_coxa_link_to_rb_femur_link: limit lower=-1.85 upper=1.57 effort=5.0 velocity=12 -> lower=-3.141592653589793 upper=3.141592653589793 effort=0.2 velocity=11.6
- joint rb_femur_link_to_rb_tibia_link: limit lower=-2.0 upper=2.75 effort=5.0 velocity=12 -> lower=-3.141592653589793 upper=3.141592653589793 effort=0.2 velocity=11.6
- joint rf_coxa_joint: limit lower=-1.0 upper=1.0 effort=5.0 velocity=12 -> lower=-3.141592653589793 upper=3.141592653589793 effort=0.2 velocity=11.6
- joint rf_coxa_link_to_rf_femur_link: limit lower=-1.85 upper=1.57 effort=5.0 velocity=12 -> lower=-3.141592653589793 upper=3.141592653589793 effort=0.2 velocity=11.6
- joint rf_femur_link_to_rf_tibia_link: limit lower=-2.0 upper=2.75 effort=5.0 velocity=12 -> lower=-3.141592653589793 upper=3.141592653589793 effort=0.2 velocity=11.6
- joint rm_coxa_joint: limit lower=-1.0 upper=1.0 effort=5.0 velocity=12 -> lower=-3.141592653589793 upper=3.141592653589793 effort=0.2 velocity=11.6
- joint rm_coxa_link_to_rm_femur_link: limit lower=-1.85 upper=1.57 effort=5.0 velocity=12 -> lower=-3.141592653589793 upper=3.141592653589793 effort=0.2 velocity=11.6
- joint rm_femur_link_to_rm_tibia_link: limit lower=-2.0 upper=2.75 effort=5.0 velocity=12 -> lower=-3.141592653589793 upper=3.141592653589793 effort=0.2 velocity=11.6
